File: pcb/name_card_keyboard.kicad_pcb (KiCad board)
At the start: 2 copper layers, 91.5 x 55.9 mm, 36 parts, among them J1 USB_C_Receptacle, J2 Conn_01x12_Female, J3 Conn_01x12_Female, J4 Conn_01x06_Female, SW1 SW_Push, SW2 SW_Push, SW3 SW_Push, SW4 SW_Push, U1 ATmega32U4-AU, Y1 16MHz

Commit message: [change]change AW
Routing:
- net +5V: track 103.1 -> 106.9 mm
- net GNDPWR: track 85.8 -> 88.6 mm, vias 81 -> 85
- net /A3: track 109.3 -> 111.5 mm
- net /A2: track 120.5 -> 121.9 mm
- net Net-(D2-Pad2): track 8.22 -> 7.52 mm
- net /A0: track 53.0 -> 52.4 mm

Commit message: [change]update pcb
Parts:
- removed the G*** at (112.8, 90.2)
- added G***: LOGO, name_card_keyboard:logo_study_in_scarlet, F.Cu at (135.9, 132.1)
- added G***: LOGO, name_card_keyboard:qr_code, F.Cu at (107.3, 95.2)
- F1: value 5A 13.2V 1608 -> NANOSMDC050F/13.2; footprint Fuse:Fuse_0603_1608Metric -> Fuse:Fuse_1206_3216Metric
- J1: value USB_C_Receptacle -> CX70M-24P1
- moved R5 14.6 mm to (186.8, 88.3)
- moved C5 9.92 mm to (172.7, 90.8)
- moved D2 9.86 mm to (186.8, 90.8)
- moved R2 8.26 mm to (178.4, 101.0)
- moved D1 7.47 mm to (179.1, 86.4), turned to 180 degrees
- moved J1 6.98 mm to (184.3, 99.7)
- moved C2 6.84 mm to (178.6, 92.7)
- moved R1 5.72 mm to (178.4, 103.5)
- moved C1 5.72 mm to (153.8, 82.5)
- moved C3 5.72 mm to (164.0, 82.5), turned to 180 degrees
- moved C6 5.72 mm to (171.6, 105.9)
- moved C7 5.72 mm to (172.8, 97.8)
- moved D4 5.72 mm to (134.7, 102.9)
- moved D5 5.72 mm to (141.1, 102.9)
- moved D6 5.72 mm to (147.4, 102.9)
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Connections:
- J3 pad 1: VCC -> +5V
- J3 pad 4: VCC -> +5V
- R2 pad 1: /D+ -> /D-
- R4 pad 1: /D- -> /D+
- U1 pad 33: Net-(U1-Pad33) -> GNDPWR
Routing:
- net VCC: track 145.5 -> 56.0 mm, vias 6 -> 4
- net +5V: track 106.9 -> 57.8 mm
- net Net-(D3-Pad2): track 21.9 -> 33.7 mm
- net /D-: track 20.8 -> 9.38 mm
- net /D+: track 20.5 -> 9.46 mm
- net GNDPWR: track 88.6 -> 81.7 mm, vias 85 -> 74
- net /SCK: track 72.1 -> 65.1 mm, vias 2 -> 0
- net /A2: track 121.9 -> 116.2 mm
- net /MOSI: track 64.7 -> 59.3 mm, vias 2 -> 1
- net Net-(D5-Pad2): track 31.3 -> 26.1 mm
- net Net-(D6-Pad2): track 46.6 -> 41.4 mm
- net /A3: track 111.5 -> 116.1 mm
- net Net-(D2-Pad2): track 7.52 -> 3.78 mm
- net /MISO: track 71.4 -> 67.7 mm, vias 0 -> 1
- net Net-(J1-PadA6): track 12.7 -> 9.41 mm, vias 1 -> 2
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- added copper zone on B.Cu, net +5V
- added copper zone on F.Cu, net +5V
Other:
- outline, holes or cut-outs redrawn
- board text added: "1"
- board text added: "10"
- board text added: "14"
- board text added: "15"
- board text added: "16"
- board text added: "2"
- board text added: "20"
- board text added: "3"
- board text added: "30"
- board text added: "4"
- board text added: "40"
- board text added: "5"
- board text added: "5V"
- board text added: "6"
- board text added: "7"
- board text added: "8"
- board text added: "9"
- board text added: "A0"
- board text added: "A1"
- board text added: "A2"
- board text added: "A3"
- board text added: "GND"
- board text added: "ICSP"
- board text added: "K"
- board text added: "MISO"
- board text added: "MOSI"
- board text added: "NCK-4-20-C"
- board text added: "RAW"
- board text added: "RST"
- board text added: "RXI"
- board text added: "SCK"
- board text added: "TXO"
- board text added: "VCC"
- board text added: "https://git.io/tomskey4"
- board text removed: "THE STUDY IN SCARLET NCK-4-20-C"
- board text removed: "https://github.com/toms74209200/Name_card_Keyboard_4"
